File: PCB/PCB-DRONE.kicad_pcb (KiCad board)
At the start: 2 copper layers, 150 x 130 mm, 67 parts, among them J1 USB_C_Receptacle_USB2.0_16P, J2 Conn_01x02_Pin, M1 Motor_DC, M2 Motor_DC, M3 Motor_DC, M4 Motor_DC, Q1 AO3401A, Q2 AO3400A, Q3 AO3400A, Q4 AO3400A, Q5 AO3400A, SW1 SW_Push, SW2 SW_Push, U1 MT3608, U2 AP63203WU, U3 MPU-6050, U4 BMP280, U5 ESP32-S3-WROOM-1

Commit message: Add files via upload
Parts:
- removed C1: 2u2, Capacitor_SMD:C_0201_0603Metric
- removed R5: 100R, Resistor_SMD:R_0603_1608Metric
- added D8: 1N4001, Diode_THT:D_DO-41_SOD81_P5.08mm_Vertical_KathodeUp, F.Cu at (153.4, 104.8)
- added L1: 2.2uh, Inductor_SMD:L_0201_0603Metric, F.Cu at (151.9, 107.0)
- added L2: 4.7uf, Inductor_SMD:L_0603_1608Metric, F.Cu at (160.5, 99.9)
- C15, C16, C7, C8: value C -> 50nf
- C2: value 2u2 -> 47uf
- C3: value 2u2 -> 10uf
- C4: value 100n -> 100nf
- C6: value 100n -> 22uf
- moved F1 0.73 mm to (153.4, 107.3), turned to 180 degrees
Connections:
- U2 pad 1: 3.3V -> Net-(U2-FB)
Routing:
- net Net-(D8-K): track 8.46 -> 12.2 mm
- net Net-(U2-FB): track 0.00 -> 2.98 mm
- net 3.3V: track 96.4 -> 98.8 mm
- net GND: track 210.6 -> 209.8 mm
Other:
- board size 150 x 130 mm -> 148.3 x 128.3 mm
