File: PCB/PCB-DRONE.kicad_sch (KiCad schematic)
At the start: 67 parts, among them J1 USB_C_Receptacle_USB2.0_16P, J2 Conn_01x02_Pin, M1 Motor_DC, M2 Motor_DC, M3 Motor_DC, M4 Motor_DC, Q1 AO3401A, Q2 AO3400A, Q3 AO3400A, Q4 AO3400A, Q5 AO3400A, SW1 SW_Push, SW2 SW_Push, U1 MT3608, U2 AP63203WU, U3 MPU-6050, U4 BMP280, U5 ESP32-S3-WROOM-1

Commit message: Add files via upload
Parts:
- removed C1: 2u2, Capacitor_SMD:C_0201_0603Metric, symbol Device:C
- removed R5: 100R, Resistor_SMD:R_0603_1608Metric, symbol Device:R
- added D8: 1N4001, Diode_THT:D_DO-41_SOD81_P5.08mm_Vertical_KathodeUp, symbol Diode:1N4001
- added L1: 2.2uh, Inductor_SMD:L_0201_0603Metric, symbol Device:L
- added L2: 4.7uf, Inductor_SMD:L_0603_1608Metric, symbol Device:L
- C15, C16, C7, C8: value C -> 50nf
- C2: value 2u2 -> 47uf
- C3: value 2u2 -> 10uf
- C4: value 100n -> 100nf
- C6: value 100n -> 22uf
Connections:
- net 3.3V: now also L2.1; no longer U2.1 (FB)
- net GND: now also D8.2 (A)
- net at C2.1, C3.1, U2.2 (EN)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: now also D8.1 (K), L1.2
- net at F1.2: now also L1.1
- new net: L2.2, U2.1 (FB)
Other:
- moved on the sheet: C18, C19, U1
